Commit message: Add aligned_depth_to_color topic for rtabmap

File: urdf/raspicat.urdf.xacro (robot description, xacro)
@@ -104,5 +104,5 @@
     <xacro:if value="$(arg camera_gazebo_plugin)">
       <xacro:realsensed435_color_gazebo
-        color_fps="15" color_width="1920" color_height="1080"/>
+        color_fps="15" color_width="1920" color_height="1080" pointCloud_z_min="0.2" pointCloud_z_max="5"/>
       <xacro:realsensed435_depth_gazebo
         depth_fps="15" depth_width="1280" depth_height="720" pointCloud_z_min="0.2" pointCloud_z_max="5"/>

File: urdf/sensors/realsense_d435.gazebo.xacro (robot description, xacro)
@@ -1,9 +1,9 @@
 <?xml version="1.0"?>
 <robot xmlns:xacro="http://ros.org/wiki/xacro">
-  <xacro:macro name="realsensed435_color_gazebo" params="color_fps color_width color_height">
+  <xacro:macro name="realsensed435_color_gazebo" params="color_fps color_width color_height pointCloud_z_min pointCloud_z_max">
     <gazebo reference="camera_color_frame">
-      <sensor type="camera" name="color_camera">
+      <sensor type="depth" name="color_camera">
         <update_rate>${color_fps}</update_rate>
-        <camera name="color_camera">
+        <camera name="color_and_aligned_depth_camera">
           <horizontal_fov>${radians(69.4)}</horizontal_fov>
           <image>
@@ -13,15 +13,20 @@
           </image>
           <clip>
-            <near>0.02</near>
-            <far>300.0</far>
+            <near>${pointCloud_z_min}</near>
+            <far>${pointCloud_z_max}</far>
           </clip>
         </camera>
-        <plugin name="color_camera_controller" filename="libgazebo_ros_camera.so">
+        <plugin name="color_and_aligned_depth_camera" filename="libgazebo_ros_openni_kinect.so">
           <baseline>0.2</baseline>
           <alwaysOn>true</alwaysOn>
           <updateRate>${color_fps}</updateRate>
-          <cameraName>camera/color</cameraName>
-          <imageTopicName>image_raw</imageTopicName>
-          <cameraInfoTopicName>camera_info</cameraInfoTopicName>
+          <cameraName>camera</cameraName>
+          <depthImageTopicName>aligned_depth_to_color/image_raw</depthImageTopicName>
+          <depthImageCameraInfoTopicName>aligned_depth_to_color/camera_info</depthImageCameraInfoTopicName>
+          <imageTopicName>color/image_raw</imageTopicName>
+          <cameraInfoTopicName>color/camera_info</cameraInfoTopicName>
+          <pointCloudTopicName>aligned_depth_to_color/points</pointCloudTopicName>
+          <pointCloudCutoff>${pointCloud_z_min}</pointCloudCutoff>
+          <pointCloudCutoffMax>${pointCloud_z_max}</pointCloudCutoffMax>
           <frameName>camera_color_optical_frame</frameName>
           <hackBaseline>0.07</hackBaseline>
@@ -56,5 +61,5 @@
           <updateRate>${depth_fps}</updateRate>
           <cameraName>camera/depth</cameraName>
-          <depthImageTopicName>image_raw</depthImageTopicName>
+          <depthImageTopicName>image_rect_raw</depthImageTopicName>
           <depthImageCameraInfoTopicName>camera_info</depthImageCameraInfoTopicName>
           <imageTopicName>color/image_raw</imageTopicName>

File: urdf/sensors/realsense_d435.urdf.xacro (robot description, xacro)
@@ -16,5 +16,5 @@
     <link name="camera_color_frame"/>
     <joint name="camera_color_optical_joint" type="fixed">
-      <origin xyz="0 0 0" rpy="0 0 0"/>
+      <origin xyz="0 0 0" rpy="${-M_PI/2} 0 ${-M_PI/2}"/>
       <parent link="camera_color_frame"/>
       <child link="camera_color_optical_frame"/>
